File: Project Architecture.kicad_sch (KiCad schematic)
At the start: 0 parts

Commit message: started migration
Parts:
- added H701, H702, H703, H704, H705, H706, H707, H708: MountingHole, MountingHole:MountingHole_3.2mm_M3, symbol Mechanical:MountingHole
- added J701: ZHOURI DC3, Connector_IDC:IDC-Header_2x05_P2.54mm_Horizontal, symbol Connector_Generic:Conn_02x05_Odd_Even
- added JP701: 0R, Resistor_THT:R_Axial_DIN0204_L3.6mm_D1.6mm_P5.08mm_Horizontal, symbol Device:R
- added P701, P702, P703: ~, symbol personal:Cosmetic_PWR
- added P704, P705: ~, symbol personal:Cosmetic_GND2
- added R701: 10k, Resistor_SMD:R_0603_1608Metric_Pad0.98x0.95mm_HandSolder, symbol Device:R
Connections:
- new net: J701.2 (Pin_2), JP701.1
- new net Earth: JP701.2
- new net GND: J701.5 (Pin_5), P704.1, P705.1
- new net SL3: J701.6 (Pin_6), P701.1, P702.1, P703.1, R701.1
- new net Section A - Title A/LV_NRST: J701.9 (Pin_9), R701.2
- new net Section A - Title A/LV_RX: J701.1 (Pin_1)
- new net Section A - Title A/LV_SWDCLK: J701.10 (Pin_10)
- new net Section A - Title A/LV_SWDIO: J701.8 (Pin_8)
- new net Section A - Title A/LV_TX: J701.3 (Pin_3)
- no-connect marks 0 -> 2
Other:
- removed sheet Section B - Title B
- sheet Section A - Title A ports: added Earth, GND, LV_NRST, LV_RX, LV_SWDCLK, LV_SWDIO, LV_TX, SL3; removed none
- note removed: "Page 5"
