File: Section A - Title A.kicad_sch (KiCad schematic)
At the start: 0 parts

Commit message: started migration
Parts:
- added C701, C702, C703, C704, C705, C708, C709, C710, C713: 100n, Capacitor_SMD:C_0603_1608Metric_Pad1.08x0.95mm_HandSolder, symbol Device:C
- added C706, C707: 1u, Capacitor_SMD:C_0603_1608Metric_Pad1.08x0.95mm_HandSolder, symbol Device:C
- added C711, C712: 22p, Capacitor_SMD:C_0603_1608Metric_Pad1.08x0.95mm_HandSolder, symbol Device:C
- added D701: LED, LED_THT:LED_D3.0mm, symbol Device:LED
- added D702: LED, LED_SMD:LED_PLCC-2_3x2mm_KA, symbol Device:LED
- added J702: 1050171001 Micro Type B, Personal:USB_Micro-B_Molex-105017-0001, symbol Connector:USB_B_Micro
- added J703, J704: Conn_01x04_Pin, Connector_PinSocket_2.54mm:PinSocket_1x04_P2.54mm_Vertical, symbol Connector:Conn_01x04_Pin
- added J705: Conn_01x14_Pin, Connector_PinSocket_2.54mm:PinSocket_1x14_P2.54mm_Vertical, symbol Connector:Conn_01x14_Pin
- added J706: Header, Connector_PinHeader_2.54mm:PinHeader_1x02_P2.54mm_Vertical, symbol Connector:Conn_01x02_Pin
- added J707, J708: HX JN1.27-2x5 WZ H4.9, Personal:JN1.27-2x5 WZ H4.9, symbol Connector_Generic:Conn_02x05_Odd_Even
- added JP702, JP704, JP705, JP706, JP707, JP709, JP711, JP712, JP716: 0R, Resistor_SMD:R_0603_1608Metric_Pad0.98x0.95mm_HandSolder, symbol Device:R
- added JP703: 8.12, Personal:Jumper_mm_L8.12_D1.2_H0.5, symbol Jumper:Jumper_2_Bridged
- added JP708, JP715: 0R, Resistor_THT:R_Axial_DIN0204_L3.6mm_D1.6mm_P7.62mm_Horizontal, symbol Device:R
- added JP710, JP713, JP714: 0R, Resistor_THT:R_Axial_DIN0204_L3.6mm_D1.6mm_P5.08mm_Horizontal, symbol Device:R
- added OLED701: OLED_128x64_SSD1306, Personal:OLED_SSD1306_no_pins, symbol personal:OLED_128x64_SSD1306_no_pins
- added P706, P728, P729, P730, P733, P739, P749, P771, P789, P791, P792, P793, P794: ~, symbol personal:Cosmetic_PWR
- added P707: ~, symbol personal:Cosmetic_PWR_SRC
- added P708, P714, P715, P716, P745, P750, P751, P752, P753, P754, P756, P758, P763, P764, P767, P768, P790, P802, P803, P804, P805: ~, symbol personal:Cosmetic_OUT
- added P709, P712, P713, P734, P744, P746, P747, P748, P755, P757, P760, P762, P765, P766, P769, P773, P774, P776, P777, P781, P782, P784, P786, P799: ~, symbol personal:Cosmetic_IN
- added P710, P717, P718, P719, P720, P721, P722, P723, P724, P725, P726, P727, P735, P737, P738, P740, P741, P742, P743, P778, P779, P780, P783, P785, P787, P788, P795, P796, P797, P798, P806: ~, symbol personal:Cosmetic_GND2
- added P711, P731, P732, P736, P761, P770, P772, P775, P800, P801: ~, symbol personal:Cosmetic_IO
- added R702, R703, R704, R706, R707, R708, R710, R711, R712, R726: 1k, Resistor_SMD:R_0603_1608Metric_Pad0.98x0.95mm_HandSolder, symbol Device:R
- added R705, R709, R713: 220k, Resistor_SMD:R_0603_1608Metric_Pad0.98x0.95mm_HandSolder, symbol Device:R
- added R714, R715, R716: 44k, Resistor_SMD:R_0603_1608Metric_Pad0.98x0.95mm_HandSolder, symbol Device:R
- added R717, R718, R719: 22k, Resistor_SMD:R_0603_1608Metric_Pad0.98x0.95mm_HandSolder, symbol Device:R
- added R720, R721, R722: 11k, Resistor_SMD:R_0603_1608Metric_Pad0.98x0.95mm_HandSolder, symbol Device:R
- added R723, R724: 4k7, Resistor_SMD:R_0603_1608Metric_Pad0.98x0.95mm_HandSolder, symbol Device:R
- added R725, R727, R728: 10k, Resistor_SMD:R_0603_1608Metric_Pad0.98x0.95mm_HandSolder, symbol Device:R
- added SW701, SW702, SW703: EncSw, Personal:RotaryEncoderSwitch_Oblong, symbol Device:RotaryEncoder_Switch
- added TFT701: TFT_2.8in_320x240, Personal:TFT_2.8_IN_320x240, symbol personal:TFT_2.8_IN_320x240
- added TP701, TP702, TP703, TP704, TP705, TP706, TP707, TP708, TP709: TestPoint, TestPoint:TestPoint_THTPad_D1.0mm_Drill0.5mm, symbol Connector:TestPoint
- added U701: STM32G431K8Tx, Package_QFP:LQFP-32_7x7mm_P0.8mm, symbol MCU_ST_STM32G4:STM32G431K8Tx
- added Y701: 20 MHz, Crystal:Crystal_SMD_3225-4Pin_3.2x2.5mm_HandSoldering, symbol Device:Crystal_GND24_Small
Connections:
- new net: R703.2, R717.1, SW701.A
- new net: R702.2, R714.1, SW701.B
- new net: R704.2, R720.1, SW701.S1
- new net: J702.1 (VBUS), TP704.1
- new net: R706.2, R715.1, SW702.B
- new net: J702.2 (D-), JP706.1
- new net: J702.3 (D+), JP704.1
- new net: J702.4 (ID), TP705.1
- new net: JP715.1, U701.25 (PA15)
- new net: C701.1, JP702.1, R702.1, R703.1, R704.1, R705.1, R706.1, R707.1, R708.1, R709.1, R710.1, R711.1, R712.1, R713.1
- new net: R711.2, R719.1, SW703.A
- new net: R712.2, R722.1, SW703.S1
- new net: R707.2, R718.1, SW702.A
- new net: R710.2, R716.1, SW703.B
- new net: J705.10 (Pin_10), JP711.2
- new net: C711.1, U701.2 (PF0), Y701.1
- new net: TP706.1, U701.28 (PB5)
- new net: C712.1, U701.3 (PF1), Y701.3
- new net: J705.4 (Pin_4), JP716.2
- new net: J705.11 (Pin_11), JP710.2
- new net: JP708.2, U701.27 (PB4)
- new net: J705.12 (Pin_12), JP709.2
- new net: J705.13 (Pin_13), JP707.2
- new net: J705.5 (Pin_5), JP714.2
- new net: J705.6 (Pin_6), JP713.2
- new net: J705.9 (Pin_9), JP712.2
- new net: R708.2, R721.1, SW702.S1
- new net: D701.1 (K), D702.1 (K), R726.1
- new net BOOT0: J706.2 (Pin_2), P769.1, P790.1, R728.1, U701.31 (PB8)
- new net DISP_CS: J705.3 (Pin_3), P750.1, P786.1, U701.9 (PA4)
- new net DISP_DC: JP714.1, P751.1, P781.1, U701.13 (PB0)
- new net DISP_MISO: JP707.1, JP712.1, P755.1, P756.1, P768.1, U701.11 (PA6)
- new net DISP_MOSI: JP709.1, JP713.1, P758.1, P760.1, P776.1, U701.12 (PA7)
- new net DISP_RST: JP716.1, P767.1, P784.1, U701.20 (PA10)
- new net DISP_SCK: J705.7 (Pin_7), JP711.1, P752.1, P765.1, P774.1, U701.10 (PA5)
- new net DISP_SCL: J703.3 (Pin_3), P734.1, P764.1, R723.2, U701.19 (PA9)
- new net DISP_SDA: J703.4 (Pin_4), P731.1, P761.1, R724.2, U701.18 (PA8)
- new net Earth: J702.6 (Shield), P718.1, P740.1
- new net FREQ: C702.1, P714.1, P747.1, R705.2, R714.2, R717.2, R720.2, TP701.1, U701.7 (PA2)
- new net GND: C701.2, C702.2, C703.2, C704.2, C705.2, C706.2, C707.2, C708.2, C709.2, C710.2, C711.2, C712.2, C713.2, J702.5 (GND), J703.1 (Pin_1), J705.2 (Pin_2), J707.5 (Pin_5), J707.6 (Pin_6), J708.5 (Pin_5), J708.6 (Pin_6), P710.1, P717.1, P719.1, P720.1, P721.1, P722.1, P723.1, P724.1, P725.1, P726.1, P727.1, P735.1, P737.1, P738.1, P741.1, P742.1, P743.1, P778.1, P779.1, P780.1, P783.1, P785.1, P787.1, P788.1, P795.1, P796.1, P797.1, P798.1, P806.1, R727.2, R728.2, SW701.C, SW701.S2, SW702.C, SW702.S2, SW703.C, SW703.S2, U701.14 (VSSA), U701.16 (VSS), U701.32 (VSS), Y701.2 (G), Y701.4 (G)
- new net LV_NRST: J708.1 (Pin_1), P713.1, P804.1
- new net LV_RX: P708.1, P766.1, TP709.1, U701.30 (PB7)
- new net LV_SWDCLK: J708.2 (Pin_2), P712.1, P805.1
- new net LV_SWDIO: J708.4 (Pin_4), P711.1, P801.1
- new net LV_TX: P709.1, P763.1, TP707.1, U701.29 (PB6)
- new net NRST: J707.1 (Pin_1), P744.1, P802.1, R725.2, U701.4 (PG10)
- new net PER: C704.1, P716.1, P746.1, R713.2, R716.2, R719.2, R722.2, TP703.1, U701.6 (PA1)
- new net SL3: C705.1, C706.1, C710.1, C713.1, D701.2 (A), D702.2 (A), J703.2 (Pin_2), J705.1 (Pin_1), J705.8 (Pin_8), J706.1 (Pin_1), J707.7 (Pin_7), J707.8 (Pin_8), J708.7 (Pin_7), J708.8 (Pin_8), JP702.2, JP703.2 (B), P706.1, P707.1, P728.1, P729.1, P730.1, P733.1, P739.1, P749.1, P771.1, P789.1, P791.1, P792.1, P793.1, P794.1, R723.1, R724.1, R725.1, U701.1 (VDD)
- new net SL3_A: C709.1, JP705.2, U701.15 (VDDA)
- new net SL3_J: C707.1, C708.1, JP703.1 (A), JP705.1, U701.17 (VDD)
- new net ST_LED: P745.1, P773.1, R726.2, R727.1, TP708.1, U701.5 (PA0)
- new net SUP: C703.1, P715.1, P748.1, R709.2, R715.2, R718.2, R721.2, TP702.1, U701.8 (PA3)
- new net SWDCLK: J707.2 (Pin_2), P777.1, P803.1, U701.24 (PA14)
- new net SWDIO: J707.4 (Pin_4), P775.1, P800.1, U701.23 (PA13)
- new net SWO: J707.3 (Pin_3), P754.1, P799.1, U701.26 (PB3)
- new net TCH_CS: JP710.1, JP715.2, P762.1, P782.1
- new net TCH_IRQ: J705.14 (Pin_14), JP708.1, P753.1, P757.1
- new net USB_DM: JP706.2, P736.1, P770.1, U701.21 (PA11)
- new net USB_DP: JP704.2, P732.1, P772.1, U701.22 (PA12)
- no-connect marks 0 -> 9
Other:
- note added: "3D model"
- note added: "BLOCK INTERFACE"
- note added: "Boot config"
- note added: "Encoder interface"
- note added: "HMI 700"
- note added: "HMI microcontroller"
- note added: "OLED display"
- note added: "SWD header - HMI"
- note added: "SWD header - Main"
- note added: "Status LED"
- note added: "TFT display"
- note added: "USB interface (serial comms port)"
