File: Strobe_HMI.kicad_pcb (KiCad board)
At the start: 6 copper layers, 0 parts

Commit message: started migration
Parts:
- added C701: 100n, Capacitor_SMD:C_0603_1608Metric_Pad1.08x0.95mm_HandSolder, F.Cu at (408.5, 120.0)
- added C702: 100n, Capacitor_SMD:C_0603_1608Metric_Pad1.08x0.95mm_HandSolder, F.Cu at (389.0, 101.1)
- added C703: 100n, Capacitor_SMD:C_0603_1608Metric_Pad1.08x0.95mm_HandSolder, F.Cu at (389.0, 67.1)
- added C704: 100n, Capacitor_SMD:C_0603_1608Metric_Pad1.08x0.95mm_HandSolder, F.Cu at (389.0, 135.1)
- added C705: 100n, Capacitor_SMD:C_0603_1608Metric_Pad1.08x0.95mm_HandSolder, F.Cu at (350.6, 93.9)
- added C706: 1u, Capacitor_SMD:C_0603_1608Metric_Pad1.08x0.95mm_HandSolder, F.Cu at (352.2, 94.5)
- added C707: 1u, Capacitor_SMD:C_0603_1608Metric_Pad1.08x0.95mm_HandSolder, F.Cu at (340.4, 80.6)
- added C708: 100n, Capacitor_SMD:C_0603_1608Metric_Pad1.08x0.95mm_HandSolder, F.Cu at (340.4, 83.9)
- added C709: 100n, Capacitor_SMD:C_0603_1608Metric_Pad1.08x0.95mm_HandSolder, F.Cu at (343.8, 82.1)
- added C710: 100n, Capacitor_SMD:C_0603_1608Metric_Pad1.08x0.95mm_HandSolder, F.Cu at (368.0, 79.1)
- added C711: 22p, Capacitor_SMD:C_0603_1608Metric_Pad1.08x0.95mm_HandSolder, F.Cu at (356.3, 95.1)
- added C712: 22p, Capacitor_SMD:C_0603_1608Metric_Pad1.08x0.95mm_HandSolder, F.Cu at (359.9, 91.9)
- added C713: 100n, Capacitor_SMD:C_0603_1608Metric_Pad1.08x0.95mm_HandSolder, F.Cu at (364.9, 53.0)
- added D701: LED, LED_THT:LED_D3.0mm, F.Cu at (365.3, 139.5)
- added D702: LED, LED_SMD:LED_PLCC-2_3x2mm_KA, F.Cu at (369.1, 140.8)
- added H701: MountingHole, MountingHole:MountingHole_3.2mm_M3, F.Cu at (407.7, 51.6)
- added H702: MountingHole, MountingHole:MountingHole_3.2mm_M3, F.Cu at (317.7, 51.6)
- added H703: MountingHole, MountingHole:MountingHole_3.2mm_M3, F.Cu at (407.7, 141.6)
- added H704: MountingHole, MountingHole:MountingHole_3.2mm_M3, F.Cu at (359.6, 105.3)
- added H705: MountingHole, MountingHole:MountingHole_3.2mm_M3, F.Cu at (401.7, 79.6)
- added H706: MountingHole, MountingHole:MountingHole_3.2mm_M3, F.Cu at (317.7, 141.6)
- added H707: MountingHole, MountingHole:MountingHole_3.2mm_M3, F.Cu at (380.7, 105.4)
- added H708: MountingHole, MountingHole:MountingHole_3.2mm_M3, F.Cu at (401.7, 113.6)
- added J701: ZHOURI DC3, Connector_IDC:IDC-Header_2x05_P2.54mm_Horizontal, F.Cu at (338.2, 121.8)
- added J702: 1050171001 Micro Type B, Personal:USB_Micro-B_Molex-105017-0001, F.Cu at (315.5, 60.9)
- added J703: Conn_01x04_Pin, Connector_PinSocket_2.54mm:PinSocket_1x04_P2.54mm_Vertical, F.Cu at (366.4, 81.6)
- added J704: Conn_01x04_Pin, Connector_PinSocket_2.54mm:PinSocket_1x04_P2.54mm_Vertical, F.Cu at (353.6, 134.2)
- added J705: Conn_01x14_Pin, Connector_PinSocket_2.54mm:PinSocket_1x14_P2.54mm_Vertical, F.Cu at (366.3, 56.0)
- added J706: Header, Connector_PinHeader_2.54mm:PinHeader_1x02_P2.54mm_Vertical, F.Cu at (354.2, 141.4)
- added J707: HX JN1.27-2x5 WZ H4.9, Personal:JN1.27-2x5 WZ H4.9, F.Cu at (320.9, 78.3)
- added J708: HX JN1.27-2x5 WZ H4.9, Personal:JN1.27-2x5 WZ H4.9, F.Cu at (320.9, 97.4)
- added JP701: 0R, Resistor_THT:R_Axial_DIN0204_L3.6mm_D1.6mm_P5.08mm_Horizontal, F.Cu at (334.9, 128.9)
- added JP702: 0R, Resistor_SMD:R_0603_1608Metric_Pad0.98x0.95mm_HandSolder, F.Cu at (408.5, 118.5)
- added JP703: 8.12, Personal:Jumper_mm_L8.12_D1.2_H0.5, F.Cu at (348.3, 77.2)
- added JP704: 0R, Resistor_SMD:R_0603_1608Metric_Pad0.98x0.95mm_HandSolder, F.Cu at (322.2, 61.3)
- added JP705: 0R, Resistor_SMD:R_0603_1608Metric_Pad0.98x0.95mm_HandSolder, F.Cu at (340.4, 82.2)
- added JP706: 0R, Resistor_SMD:R_0603_1608Metric_Pad0.98x0.95mm_HandSolder, F.Cu at (322.2, 59.8)
- added JP707: 0R, Resistor_SMD:R_0603_1608Metric_Pad0.98x0.95mm_HandSolder, F.Cu at (335.9, 61.0)
- added JP708: 0R, Resistor_THT:R_Axial_DIN0204_L3.6mm_D1.6mm_P7.62mm_Horizontal, F.Cu at (335.0, 86.4)
- added JP709: 0R, Resistor_SMD:R_0603_1608Metric_Pad0.98x0.95mm_HandSolder, F.Cu at (338.4, 61.0)
- added JP710: 0R, Resistor_THT:R_Axial_DIN0204_L3.6mm_D1.6mm_P5.08mm_Horizontal, F.Cu at (341.0, 65.4)
- added JP711: 0R, Resistor_SMD:R_0603_1608Metric_Pad0.98x0.95mm_HandSolder, F.Cu at (343.5, 61.0)
- added JP712: 0R, Resistor_SMD:R_0603_1608Metric_Pad0.98x0.95mm_HandSolder, F.Cu at (346.0, 61.0)
- added JP713: 0R, Resistor_THT:R_Axial_DIN0204_L3.6mm_D1.6mm_P5.08mm_Horizontal, F.Cu at (347.4, 64.0)
- added JP714: 0R, Resistor_THT:R_Axial_DIN0204_L3.6mm_D1.6mm_P5.08mm_Horizontal, F.Cu at (347.4, 66.8)
- added JP715: 0R, Resistor_THT:R_Axial_DIN0204_L3.6mm_D1.6mm_P7.62mm_Horizontal, F.Cu at (338.7, 94.0)
- added JP716: 0R, Resistor_SMD:R_0603_1608Metric_Pad0.98x0.95mm_HandSolder, F.Cu at (348.6, 53.0)
- added OLED701: OLED_128x64_SSD1306, Personal:OLED_SSD1306_no_pins, F.Cu at (370.2, 93.8)
- added R701: 10k, Resistor_SMD:R_0603_1608Metric_Pad0.98x0.95mm_HandSolder, F.Cu at (328.0, 100.5)
- added R702: 1k, Resistor_SMD:R_0603_1608Metric_Pad0.98x0.95mm_HandSolder, F.Cu at (389.0, 96.6)
- added R703: 1k, Resistor_SMD:R_0603_1608Metric_Pad0.98x0.95mm_HandSolder, F.Cu at (389.0, 93.6)
- added R704: 1k, Resistor_SMD:R_0603_1608Metric_Pad0.98x0.95mm_HandSolder, F.Cu at (389.0, 90.6)
- added R705: 220k, Resistor_SMD:R_0603_1608Metric_Pad0.98x0.95mm_HandSolder, F.Cu at (389.0, 99.6)
- added R706: 1k, Resistor_SMD:R_0603_1608Metric_Pad0.98x0.95mm_HandSolder, F.Cu at (389.0, 62.6)
- added R707: 1k, Resistor_SMD:R_0603_1608Metric_Pad0.98x0.95mm_HandSolder, F.Cu at (389.0, 59.6)
- added R708: 1k, Resistor_SMD:R_0603_1608Metric_Pad0.98x0.95mm_HandSolder, F.Cu at (389.0, 56.6)
- added R709: 220k, Resistor_SMD:R_0603_1608Metric_Pad0.98x0.95mm_HandSolder, F.Cu at (389.0, 65.6)
- added R710: 1k, Resistor_SMD:R_0603_1608Metric_Pad0.98x0.95mm_HandSolder, F.Cu at (389.0, 130.6)
- added R711: 1k, Resistor_SMD:R_0603_1608Metric_Pad0.98x0.95mm_HandSolder, F.Cu at (389.0, 127.6)
- added R712: 1k, Resistor_SMD:R_0603_1608Metric_Pad0.98x0.95mm_HandSolder, F.Cu at (389.0, 124.6)
- added R713: 220k, Resistor_SMD:R_0603_1608Metric_Pad0.98x0.95mm_HandSolder, F.Cu at (389.0, 133.6)
- added R714: 44k, Resistor_SMD:R_0603_1608Metric_Pad0.98x0.95mm_HandSolder, F.Cu at (389.0, 98.1)
- added R715: 44k, Resistor_SMD:R_0603_1608Metric_Pad0.98x0.95mm_HandSolder, F.Cu at (389.0, 64.1)
- added R716: 44k, Resistor_SMD:R_0603_1608Metric_Pad0.98x0.95mm_HandSolder, F.Cu at (389.0, 132.1)
- added R717: 22k, Resistor_SMD:R_0603_1608Metric_Pad0.98x0.95mm_HandSolder, F.Cu at (389.0, 95.1)
- added R718: 22k, Resistor_SMD:R_0603_1608Metric_Pad0.98x0.95mm_HandSolder, F.Cu at (389.0, 61.1)
- added R719: 22k, Resistor_SMD:R_0603_1608Metric_Pad0.98x0.95mm_HandSolder, F.Cu at (389.0, 129.1)
- added R720: 11k, Resistor_SMD:R_0603_1608Metric_Pad0.98x0.95mm_HandSolder, F.Cu at (389.0, 92.1)
- added R721: 11k, Resistor_SMD:R_0603_1608Metric_Pad0.98x0.95mm_HandSolder, F.Cu at (389.0, 58.1)
- added R722: 11k, Resistor_SMD:R_0603_1608Metric_Pad0.98x0.95mm_HandSolder, F.Cu at (389.0, 126.1)
- added R723: 4k7, Resistor_SMD:R_0603_1608Metric_Pad0.98x0.95mm_HandSolder, F.Cu at (371.5, 78.0)
- added R724: 4k7, Resistor_SMD:R_0603_1608Metric_Pad0.98x0.95mm_HandSolder, F.Cu at (374.1, 78.0)
- added R725: 10k, Resistor_SMD:R_0603_1608Metric_Pad0.98x0.95mm_HandSolder, F.Cu at (330.0, 100.5)
- added R726: 1k, Resistor_SMD:R_0603_1608Metric_Pad0.98x0.95mm_HandSolder, F.Cu at (365.2, 124.0)
- added R727: 10k, Resistor_SMD:R_0603_1608Metric_Pad0.98x0.95mm_HandSolder, F.Cu at (366.9, 124.0)
- added R728: 10k, Resistor_SMD:R_0603_1608Metric_Pad0.98x0.95mm_HandSolder, F.Cu at (348.6, 95.7)
- added SW701: EncSw, Personal:RotaryEncoderSwitch_Oblong, F.Cu at (401.7, 96.6)
- added SW702: EncSw, Personal:RotaryEncoderSwitch_Oblong, F.Cu at (401.7, 62.6)
- added SW703: EncSw, Personal:RotaryEncoderSwitch_Oblong, F.Cu at (401.7, 130.6)
- added TFT701: TFT_2.8in_320x240, Personal:TFT_2.8_IN_320x240, F.Cu at (349.8, 95.4)
- added TP701: TestPoint, TestPoint:TestPoint_THTPad_D1.0mm_Drill0.5mm, F.Cu at (389.0, 104.3)
- added TP702: TestPoint, TestPoint:TestPoint_THTPad_D1.0mm_Drill0.5mm, F.Cu at (389.0, 70.2)
- added TP703: TestPoint, TestPoint:TestPoint_THTPad_D1.0mm_Drill0.5mm, F.Cu at (389.0, 138.0)
- added TP704: TestPoint, TestPoint:TestPoint_THTPad_D1.0mm_Drill0.5mm, F.Cu at (319.7, 56.7)
- added TP705: TestPoint, TestPoint:TestPoint_THTPad_D1.0mm_Drill0.5mm, F.Cu at (319.7, 64.9)
- added TP706: TestPoint, TestPoint:TestPoint_THTPad_D1.0mm_Drill0.5mm, F.Cu at (343.7, 102.2)
- added TP707: TestPoint, TestPoint:TestPoint_THTPad_D1.0mm_Drill0.5mm, F.Cu at (344.0, 112.6)
- added TP708: TestPoint, TestPoint:TestPoint_THTPad_D1.0mm_Drill0.5mm, F.Cu at (366.3, 112.6)
- added TP709: TestPoint, TestPoint:TestPoint_THTPad_D1.0mm_Drill0.5mm, F.Cu at (348.1, 116.0)
- added U701: STM32G431K8Tx, Package_QFP:LQFP-32_7x7mm_P0.8mm, F.Cu at (346.4, 88.4)
- added Y701: 20 MHz, Crystal:Crystal_SMD_3225-4Pin_3.2x2.5mm_HandSoldering, F.Cu at (356.3, 91.9)
Routing:
- net /SL3: track 0.00 -> 470.9 mm
- net Net-(C701-Pad1): track 0.00 -> 180.0 mm
- net /700 HMI/PER: track 0.00 -> 88.9 mm
- net Earth: track 0.00 -> 84.4 mm
- net /700 HMI/SUP: track 0.00 -> 66.1 mm
- net /700 HMI/FREQ: track 0.00 -> 59.9 mm
- net /700 HMI/DISP_RST: track 0.00 -> 59.2 mm
- net /700 HMI/NRST: track 0.00 -> 53.5 mm, vias 0 -> 2
- net /700 HMI/BOOT0: track 0.00 -> 52.2 mm
- net /700 HMI/ST_LED: track 0.00 -> 50.0 mm
- net /700 HMI/USB_DM: track 0.00 -> 42.7 mm
- net /700 HMI/USB_DP: track 0.00 -> 42.7 mm
- net /700 HMI/SWO: track 0.00 -> 39.8 mm
- net /GND: track 0.00 -> 38.4 mm, vias 0 -> 15
- net /700 HMI/DISP_MISO: track 0.00 -> 38.2 mm
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- added copper zone on B.Cu, net /GND
Other:
- board outline added: 100 x 100 mm
- board text added: "Boot 0 Fitted -> HI Not fitted -> Lo"
- board text added: "COM port (type B micro USB)"
- board text added: "Felipe L. Rodrigues"
- board text added: "Frequency (PA2)"
- board text added: "HMI SWD"
- board text added: "HMI board"
- board text added: "HMI board Rev.1 06/09/2025 Felipe L. Rodrigues"
- board text added: "MAIN BOARD INTERFACE"
- board text added: "MAIN SWD"
- board text added: "Period (PA1)"
- board text added: "Rev.1 06/09/2025"
- board text added: "Status (PA0)"
- board text added: "Supply (PA3)"
