File: Strobe_HMI.kicad_pcb (KiCad board)
At the start: 6 copper layers, 100 x 100 mm, 91 parts, among them J701 ZHOURI DC3, J702 1050171001 Micro Type B, J703 Conn_01x04_Pin, J704 Conn_01x04_Pin, J705 Conn_01x14_Pin, J706 Header, J707 HX JN1.27-2x5 WZ H4.9, J708 HX JN1.27-2x5 WZ H4.9, SW701 EncSw, SW702 EncSw, SW703 EncSw, U701 STM32G431K8Tx, Y701 20 MHz

Commit message: sch refactoring complete
Connections:
- net /700 HMI/BOOT0 renamed /Block diagram/HMI/BOOT0
- net /700 HMI/DISP_CS renamed /Block diagram/HMI/DISP_CS
- net /700 HMI/DISP_DC renamed /Block diagram/HMI/DISP_DC
- net /700 HMI/DISP_MISO renamed /Block diagram/HMI/DISP_MISO
- net /700 HMI/DISP_MOSI renamed /Block diagram/HMI/DISP_MOSI
- net /700 HMI/DISP_RST renamed /Block diagram/HMI/DISP_RST
- net /700 HMI/DISP_SCK renamed /Block diagram/HMI/DISP_SCK
- net /700 HMI/DISP_SCL renamed /Block diagram/HMI/DISP_SCL
- net /700 HMI/DISP_SDA renamed /Block diagram/HMI/DISP_SDA
- net /700 HMI/FREQ renamed /Block diagram/HMI/FREQ
- net /700 HMI/LV_NRST renamed /Block diagram/HMI/LV_NRST
- net /700 HMI/LV_RX renamed /Block diagram/HMI/LV_RX
- net /700 HMI/LV_SWDCLK renamed /Block diagram/HMI/LV_SWDCLK
- net /700 HMI/LV_SWDIO renamed /Block diagram/HMI/LV_SWDIO
- net /700 HMI/LV_TX renamed /Block diagram/HMI/LV_TX
- net /700 HMI/NRST renamed /Block diagram/HMI/NRST
- net /700 HMI/PER renamed /Block diagram/HMI/PER
- net /700 HMI/SL3_A renamed /Block diagram/HMI/SL3_A
- net /700 HMI/SL3_J renamed /Block diagram/HMI/SL3_J
- net /700 HMI/ST_LED renamed /Block diagram/HMI/ST_LED
- net /700 HMI/SUP renamed /Block diagram/HMI/SUP
- net /700 HMI/SWDCLK renamed /Block diagram/HMI/SWDCLK
- net /700 HMI/SWDIO renamed /Block diagram/HMI/SWDIO
- net /700 HMI/SWO renamed /Block diagram/HMI/SWO
- net /700 HMI/TCH_CS renamed /Block diagram/HMI/TCH_CS
- net /700 HMI/TCH_IRQ renamed /Block diagram/HMI/TCH_IRQ
- net /700 HMI/USB_DM renamed /Block diagram/HMI/USB_DM
- net /700 HMI/USB_DP renamed /Block diagram/HMI/USB_DP
- net /GND renamed ~
- net /SL3 renamed /Block diagram/HMI/SL3
Other:
- copper layers 6 -> 2

Commit message: Migrated PCB file to template, switched to preliminary
Parts:
- moved C705 152.8 mm to (197.8, 97.2)
- moved C712 152.8 mm to (207.2, 95.2)
- moved J704 152.8 mm to (200.9, 137.6)
- moved JP701 152.8 mm to (182.1, 132.3)
- moved JP704 152.8 mm to (169.5, 64.6)
- moved JP706 152.8 mm to (169.5, 63.1)
- moved JP715 152.8 mm to (185.9, 97.3)
- moved R701 152.8 mm to (175.3, 103.8)
- moved R724 152.8 mm to (221.3, 81.4)
- moved R728 152.8 mm to (195.8, 99.0)
- moved TP707 152.8 mm to (191.3, 116.0)
- moved C701 152.8 mm to (255.8, 123.4)
- moved C702 152.8 mm to (236.2, 104.5)
- moved C703 152.8 mm to (236.2, 70.5)
- moved C704 152.8 mm to (236.2, 138.5)
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Connections:
- net ~ renamed GND
Other:
- board text removed: "30°"
- board text removed: "3× 120°"
- board text removed: "All dimensions are in millimeters unless otherwise specified."
