File: Strobe_HMI.kicad_pcb (KiCad board)
At the start: 2 copper layers, 100 x 100 mm, 91 parts, among them J701 ZHOURI DC3, J702 1050171001 Micro Type B, J703 Conn_01x04_Pin, J704 Conn_01x04_Pin, J705 Conn_01x14_Pin, J706 Header, J707 HX JN1.27-2x5 WZ H4.9, J708 HX JN1.27-2x5 WZ H4.9, SW701 EncSw, SW702 EncSw, SW703 EncSw, U701 STM32G431K8Tx, Y701 20 MHz

Commit message: Adding silk and edges to fab doc
Other:
- board text removed: "Impedance Table"

Commit message: Preparing release
Other:
- board text added: "(BOTTOM SIDE VIEW)"

Commit message: Update Outputs (release)
Other:
- board text added: "0.02mm"
- board text added: "0.07mm (2.00oz)"
- board text added: "1.48mm"
- board text added: "B.Mask"
- board text added: "B.Paste"
- board text added: "B.Silkscreen"
- board text added: "Copper"
- board text added: "Core"
- board text added: "Dielectric"
- board text added: "Direct Printing"
- board text added: "F.Mask"
- board text added: "F.Paste"
- board text added: "F.Silkscreen"
- board text added: "FR4_7628"
- board text added: "GBR"
- board text added: "Gerber"
- board text added: "L1 (Sig, PWR)"
- board text added: "L2 (Sig, PWR)"
- board text added: "Layer"
- board text added: "Legend"
- board text added: "Material"
- board text added: "Note: external layer thicknesses are specified after plating"
- board text added: "Paste Mask"
- board text added: "Signal"
- board text added: "Solder Mask"
- board text added: "Solder Resist"
- board text added: "Thickness"
- board text added: "Total thickness: 1.66mm"
- board text added: "Type"
