File: Revision History.kicad_sch (KiCad schematic)
At the start: 0 parts

Commit message: Added code, pictures, readme, updated sch size and notes, changed to checked
Changed lines of the file:
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@@
 	(text_box "[${#}] ${TITLE}"
 		(exclude_from_sim no)
-		(at 177.8 16.51 0)
+		(at 179.07 13.97 0)
 		(size 104.14 12.7)
 		(margins 4.4999 4.4999 4.4999 4.4999)
@@
 			(font
 				(face "Times New Roman")
-				(size 6.096 6.096)
+				(size 5.08 5.08)
 				(thickness 1.2)
 				(bold yes)
 				(color 0 0 194 1)
 			)
-			(justify right)
+			(justify right bottom)
 		)
 	)
