File: Strobe_HMI.kicad_sch (KiCad schematic)
At the start: 0 parts

Commit message: started migration
Other:
- removed sheet Block Diagram
- removed sheet Power - Sequencing
Changed lines of the file:
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@@
-	)
-	(sheet
-		(at 340.36 313.69)
-		(size 35.56 5.08)
-		(exclude_from_sim no)
-		(in_bom yes)
-		(on_board yes)
-		(dnp no)
-		(stroke
-			(width 0.1524)
-			(type solid)
-		)
-		(fill
-			(color 0 0 0 0.0000)
-		)
-		(property "Sheetname" "Power - Sequencing"
-			(at 340.36 312.6609 0)
-			(effects
-				(font
-					(face "Times New Roman")
-					(size 1.905 1.905)
-					(bold yes)
-					(color 0 0 0 1)
-				)
-				(justify left bottom)
-			)
-		)
-		(property "Sheetfile" "Power - Sequencing.kicad_sch"
-			(at 341.63 314.96 0)
-			(effects
-				(font
-					(face "Arial")
-					(size 1.27 1.27)
-				)
-				(justify left top)
-			)
-		)
-		(instances
-			(project "KDT_Hierarchical_KiBot"
-				(path "/f9e05184-c88b-4a88-ae9c-ab2bdb32be7c"
-					(page "6")
-				)
-			)
-		)
 	)
 	(sheet
@@
 		)
 		(instances
-			(project "KDT_Hierarchical_KiBot"
+			(project "Strobe_HMI"
 				(path "/f9e05184-c88b-4a88-ae9c-ab2bdb32be7c"
 					(page "7")
-				)
-			)
-		)
-	)
-	(sheet
-		(at 299.72 302.26)
-		(size 35.56 5.08)
-		(exclude_from_sim no)
-		(in_bom yes)
-		(on_board yes)
-		(dnp no)
-		(stroke
-			(width 0.1524)
-			(type solid)
-		)
-		(fill
-			(color 0 0 0 0.0000)
-		)
-		(property "Sheetname" "Block Diagram"
-			(at 299.72 301.2309 0)
-			(effects
-				(font
-					(face "Times New Roman")
-					(size 1.905 1.905)
-					(bold yes)
-					(color 0 0 0 1)
-				)
-				(justify left bottom)
-			)
-		)
-		(property "Sheetfile" "Block Diagram.kicad_sch"
-			(at 300.99 303.53 0)
-			(effects
-				(font
-					(face "Arial")
-					(size 1.27 1.27)
-				)
-				(justify left top)
-			)
-		)
-		(instances
-			(project "KDT_Hierarchical_KiBot"
-				(path "/f9e05184-c88b-4a88-ae9c-ab2bdb32be7c"
-					(page "2")
 				)
 			)
@@
 		)
 		(instances
-			(project "KDT_Hierarchical_KiBot"
+			(project "Strobe_HMI"
 				(path "/f9e05184-c88b-4a88-ae9c-ab2bdb32be7c"
 					(page "3")

Commit message: Refactoring sch
Other:
- sheet Project Architecture renamed Block diagram
- sheet Block diagram: file Project Architecture.kicad_sch -> Block diagram.kicad_sch
- note removed: "${SHEET_NAME_11}"
- note removed: "${SHEET_NAME_12}"
- note removed: "${SHEET_NAME_13}"
- note removed: "${SHEET_NAME_14}"
- note removed: "${SHEET_NAME_15}"
- note removed: "${SHEET_NAME_16}"
- note removed: "${SHEET_NAME_17}"
- note removed: "${SHEET_NAME_18}"
- note removed: "${SHEET_NAME_19}"
- note removed: "${SHEET_NAME_20}"
- note removed: "${SHEET_NAME_21}"
- note removed: "${SHEET_NAME_22}"
- note removed: "${SHEET_NAME_23}"
- note removed: "${SHEET_NAME_24}"
- note removed: "${SHEET_NAME_25}"
- note removed: "${SHEET_NAME_26}"
- note removed: "${SHEET_NAME_27}"
- note removed: "${SHEET_NAME_28}"
- note removed: "${SHEET_NAME_29}"
- note removed: "${SHEET_NAME_30}"
- note removed: "${SHEET_NAME_31}"
- note removed: "${SHEET_NAME_32}"
- note removed: "${SHEET_NAME_33}"
- note removed: "${SHEET_NAME_34}"
- note removed: "${SHEET_NAME_35}"
- note removed: "${SHEET_NAME_36}"
- note removed: "${SHEET_NAME_37}"
- note removed: "${SHEET_NAME_38}"
- note removed: "${SHEET_NAME_39}"
- note removed: "${SHEET_NAME_40}"
- note removed: "11"
- note removed: "12"
- note removed: "13"
- note removed: "14"
- note removed: "15"
- note removed: "16"
- note removed: "17"
- note removed: "18"
- note removed: "19"
- note removed: "20"
- note removed: "21"
- note removed: "22"
- note removed: "23"
- note removed: "24"
- note removed: "25"
- note removed: "26"
- note removed: "27"
- note removed: "28"
- note removed: "29"
- note removed: "30"
- note removed: "31"
- note removed: "32"
- note removed: "33"
- note removed: "34"
- note removed: "35"
- note removed: "36"
- note removed: "37"
- note removed: "38"
- note removed: "39"
- note removed: "40"
- note removed: "Date: ${RELEASE_DATE}"
- note removed: "STATUS CONVENTION"

Commit message: updated pcb template
Other:
- note removed: "${SHEET_NAME_10}"
- note removed: "${SHEET_NAME_5}"
- note removed: "${SHEET_NAME_6}"
- note removed: "${SHEET_NAME_7}"
- note removed: "${SHEET_NAME_8}"
- note removed: "${SHEET_NAME_9}"
- note removed: "10"
- note removed: "5"
- note removed: "6"
- note removed: "7"
- note removed: "8"
- note removed: "9"

Commit message: Added code, pictures, readme, updated sch size and notes, changed to checked
Changed lines of the file:
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@@
 	(generator "eeschema")
 	(generator_version "9.0")
-	(paper "A3")
+	(paper "A4")
 	(title_block
 		(date "2025-01-12")
@@
 	(text "Status: ${VARIANT}"
 		(exclude_from_sim no)
-		(at 398.78 53.34 0)
-		(effects
-			(font
-				(face "Times New Roman")
-				(size 10.16 10.16)
+		(at 280.67 29.21 0)
+		(effects
+			(font
+				(face "Times New Roman")
+				(size 7.62 7.62)
 				(thickness 1)
 				(bold yes)
@@
 	(text "${SHEET_NAME_2}"
 		(exclude_from_sim no)
-		(at 38.1 71.12 0)
-		(effects
-			(font
-				(face "Times New Roman")
-				(size 4 4)
+		(at 36.83 60.96 0)
+		(effects
+			(font
+				(face "Times New Roman")
+				(size 3.048 3.048)
 				(color 0 0 0 1)
 			)
@@
 	(text "Page"
 		(exclude_from_sim no)
-		(at 31.75 50.8 0)
-		(effects
-			(font
-				(face "Times New Roman")
-				(size 4 4)
+		(at 30.48 40.64 0)
+		(effects
+			(font
+				(face "Times New Roman")
+				(size 3.048 3.048)
 				(bold yes)
 				(color 0 0 0 1)
@@
 	(text "${RELEASE_DATE_NUM}"
 		(exclude_from_sim no)
-		(at 398.78 71.12 0)
-		(effects
-			(font
-				(face "Times New Roman")
-				(size 10.16 10.16)
+		(at 280.67 41.91 0)
+		(effects
+			(font
+				(face "Times New Roman")
+				(size 7.62 7.62)
 				(thickness 1)
 				(bold yes)
@@
 	(text "1"
 		(exclude_from_sim no)
-		(at 31.75 63.5 0)
-		(effects
-			(font
-				(face "Times New Roman")
-				(size 4 4)
+		(at 30.48 53.34 0)
+		(effects
+			(font
+				(face "Times New Roman")
+				(size 3.048 3.048)
 				(color 0 0 0 1)
 			)
@@
 	(text "Rev ${REVISION}"
 		(exclude_from_sim no)
-		(at 398.78 35.56 0)
-		(effects
-			(font
-				(face "Times New Roman")
-				(size 10.16 10.16)
+		(at 168.91 29.21 0)
+		(effects
+			(font
+				(face "Times New Roman")
+				(size 7.62 7.62)
 				(thickness 1)
 				(bold yes)
@@
 	(text "BOTTOM VIEW"
 		(exclude_from_sim no)
-		(at 259.08 101.6 0)
+		(at 190.5 55.88 0)
 		(effects
 			(font
@@
 	(text "2"
 		(exclude_from_sim no)
-		(at 31.75 71.12 0)
-		(effects
-			(font
-				(face "Times New Roman")
-				(size 4 4)
+		(at 30.48 60.96 0)
+		(effects
+			(font
+				(face "Times New Roman")
+				(size 3.048 3.048)
 				(color 0 0 0 1)
 			)
@@
 	(text "3"
 		(exclude_from_sim no)
-		(at 31.75 78.74 0)
-		(effects
-			(font
-				(face "Times New Roman")
-				(size 4 4)
+		(at 30.48 68.58 0)
+		(effects
+			(font
+				(face "Times New Roman")
+				(size 3.048 3.048)
 				(color 0 0 0 1)
 			)
@@
 	(text "${BOARD_NAME}"
 		(exclude_from_sim no)
-		(at 25.4 40.64 0)
-		(effects
-			(font
-				(face "Times New Roman")
-				(size 10.16 10.16)
+		(at 15.24 29.21 0)
+		(effects
+			(font
+				(face "Times New Roman")
+				(size 7.62 7.62)
 				(thickness 1)
 				(bold yes)
@@
 	(text "${SHEET_NAME_1}"
 		(exclude_from_sim no)
-		(at 38.1 63.5 0)
-		(effects
-			(font
-				(face "Times New Roman")
-				(size 4 4)
+		(at 36.83 53.34 0)
+		(effects
+			(font
+				(face "Times New Roman")
+				(size 3.048 3.048)
 				(color 0 0 0 1)
 			)
@@
 	(text "${SHEET_NAME_3}"
 		(exclude_from_sim no)
-		(at 38.1 78.74 0)
-		(effects
-			(font
-				(face "Times New Roman")
-				(size 4 4)
+		(at 36.83 68.58 0)
+		(effects
+			(font
+				(face "Times New Roman")
+				(size 3.048 3.048)
 				(color 0 0 0 1)
 			)
@@
 	(text "TOP VIEW"
 		(exclude_from_sim no)
-		(at 106.68 101.6 0)
+		(at 88.9 55.88 0)
 		(effects
 			(font
@@
 	(text "Index"
 		(exclude_from_sim no)
-		(at 38.1 50.8 0)
-		(effects
-			(font
-				(face "Times New Roman")
-				(size 4 4)
+		(at 36.83 40.64 0)
+		(effects
+			(font
+				(face "Times New Roman")
+				(size 3.048 3.048)
 				(bold yes)
 				(color 0 0 0 1)
@@
 	(text "${SHEET_NAME_4}"
 		(exclude_from_sim no)
-		(at 38.1 86.36 0)
-		(effects
-			(font
-				(face "Times New Roman")
-				(size 4 4)
+		(at 36.83 76.2 0)
+		(effects
+			(font
+				(face "Times New Roman")
+				(size 3.048 3.048)
 				(color 0 0 0 1)
 			)
@@
 	(text "4"
 		(exclude_from_sim no)
-		(at 31.75 86.36 0)
-		(effects
-			(font
-				(face "Times New Roman")
-				(size 4 4)
+		(at 30.48 76.2 0)
+		(effects
+			(font
+				(face "Times New Roman")
+				(size 3.048 3.048)
 				(color 0 0 0 1)
 			)
@@
 	(text "NOTE STYLING CONVENTION"
 		(exclude_from_sim no)
-		(at 26.67 256.54 0)
-		(effects
-			(font
-				(face "Arial")
-				(size 3.81 3.81)
+		(at 16.51 161.29 0)
+		(effects
+			(font
+				(face "Arial")
+				(size 3.048 3.048)
 				(bold yes)
 				(color 53 60 207 1)
@@
 	(text_box "DESIGN NOTE:\nExample text for cautionary design notes."
 		(exclude_from_sim no)
-		(at 101.6 260.35 0)
-		(size 31.75 19.05)
+		(at 66.04 162.56 0)
+		(size 21.59 13.97)
 		(margins 2 2 2 2)
 		(stroke
@@
 			(font
 				(face "Arial")
-				(size 2.032 2.032)
+				(size 1.524 1.524)
 				(color 0 0 0 1)
 			)
@@
 	(text_box "DESIGN NOTE:\nExample text for debug notes."
 		(exclude_from_sim no)
-		(at 63.5 260.35 0)
-		(size 31.75 19.05)
+		(at 40.64 162.56 0)
+		(size 21.59 13.97)
 		(margins 2 2 2 2)
 		(stroke
@@
 			(font
 				(face "Arial")
-				(size 2.032 2.032)
+				(size 1.524 1.524)
 				(color 0 0 0 1)
 			)
@@
 	(text_box "DESIGN NOTE:\nExample text for critical design notes."
 		(exclude_from_sim no)
-		(at 139.7 260.35 0)
-		(size 31.75 19.05)
+		(at 15.24 180.34 0)
+		(size 21.59 13.97)
 		(margins 2.25 2.25 2.25 2.25)
 		(stroke
@@
 			(font
 				(face "Arial")
-				(size 2.032 2.032)
+				(size 1.524 1.524)
 				(thickness 0.4)
 				(color 0 0 0 1)
@@
 	(text_box "LAYOUT NOTE:\nExample text for critical layout guidelines."
 		(exclude_from_sim no)
-		(at 177.8 260.35 0)
-		(size 31.75 19.05)
+		(at 40.64 180.34 0)
+		(size 21.59 13.97)
 		(margins 2.25 2.25 2.25 2.25)
 		(stroke
@@
 			(font
 				(face "Arial")
-				(size 2.032 2.032)
+				(size 1.524 1.524)
 				(thickness 0.4)
 				(color 0 0 0 1)
@@
 	(text_box "kibot_image_png_3d_viewer_angled_bottom"
 		(exclude_from_sim no)
-		(at 254 101.6 0)
-		(size 139.7 127)
+		(at 185.42 55.88 0)
+		(size 88.9 88.9)
 		(margins 1.905 1.905 1.905 1.905)
 		(stroke
@@
 	(text_box "DESIGN NOTE:\nExample text for informational design notes."
 		(exclude_from_sim no)
-		(at 25.4 260.35 0)
-		(size 31.75 19.05)
+		(at 15.24 162.56 0)
+		(size 21.59 13.97)
 		(margins 2 2 2 2)
 		(stroke
@@
 			(font
 				(face "Arial")
-				(size 2.032 2.032)
+				(size 1.524 1.524)
 				(color 0 0 0 1)
 			)
@@
 	(text_box "kibot_image_png_3d_viewer_angled_top"
 		(exclude_from_sim no)
-		(at 101.6 101.6 0)
-		(size 139.7 127)
+		(at 83.82 55.88 0)
+		(size 88.9 88.9)
 		(margins 1.905 1.905 1.905 1.905)
 		(stroke
@@
 	(polyline
 		(pts
-			(xy 38.1 53.34) (xy 92.71 53.34)
+			(xy 36.83 43.18) (xy 71.12 43.18)
 		)
 		(stroke
@@
 	(polyline
 		(pts
-			(xy 19.05 53.34) (xy 31.75 53.34)
+			(xy 21.59 43.18) (xy 30.48 43.18)
 		)
 		(stroke
@@
 	)
 	(sheet
-		(at 340.36 302.26)
+		(at 251.46 215.9)
 		(size 35.56 5.08)
 		(exclude_from_sim no)
@@
 		)
 		(property "Sheetname" "Revision History"
-			(at 340.36 300.99 0)
+			(at 251.46 214.63 0)
 			(effects
 				(font
@@
 		)
 		(property "Sheetfile" "Revision History.kicad_sch"
-			(at 340.995 303.53 0)
+			(at 252.095 217.17 0)
 			(effects
 				(font
@@
 			(project "Strobe_HMI"
 				(path "/f9e05184-c88b-4a88-ae9c-ab2bdb32be7c"
-					(page "7")
+					(page "4")
 				)
 			)
@@
 	)
 	(sheet
-		(at 299.72 302.26)
+		(at 210.82 215.9)
 		(size 35.56 5.08)
 		(exclude_from_sim no)
@@
 		)
 		(property "Sheetname" "Block diagram"
-			(at 299.72 301.2309 0)
+			(at 210.82 214.8709 0)
 			(effects
 				(font
@@
 		)
 		(property "Sheetfile" "Block diagram.kicad_sch"
-			(at 300.99 303.53 0)
+			(at 212.09 217.17 0)
 			(effects
 				(font
@@
 			(project "Strobe_HMI"
 				(path "/f9e05184-c88b-4a88-ae9c-ab2bdb32be7c"
-					(page "3")
-				)
-			)
+					(page "2")
+				)
+			)
